File: prototypes/motor-board/hardware/motor-board.sch (KiCad schematic (older format))
At the start: 22 parts, among them J1 Conn_01x02, J2 Conn_01x02, J3 Conn_01x01, J4 Conn_01x02, U1 TB67H450FNG, U2 TLV9051

Commit message: More work on motor encoder; KiCad library reorganisation
Parts:
- added J?: Conn_01x01, symbol mini-mapper:Conn_01x01
- added R? (x4): CALC, mini-mapper:R_0805, symbol mini-mapper:R
- added U?: TCST1202, symbol mini-mapper:TCST1202
- added U? (x2): LM2903, symbol Comparator:LM2903
Connections:
- net labels added: +3V3
- wire segments 82 -> 102
Other:
- note added: "1. Does the current sense amplifier need input filters?\n\n2. Does the current sense amplifier need compensation?\n\n3. What supply voltage for opamp and comparator?"
- note added: "COPY TO PROJECT LIBRARY!"
- note added: "ENCODER PULSE OUTPUT"
- note added: "HYSTERESIS\n\nCOMPARATOR SELECTION\n\nCOMPARATOR POWER"
- note added: "MOTOR DRIVER"
- note added: "MOTOR ENCODER"
- note added: "POWER"
- note removed: "Does the current sense\namplifier need input filters?\n\nDoes the current sense\namplifier need compensation?"
- moved on the sheet: C1, C2, C3, C?, J1, J2, J4, NT1, NT2, NT?, R1, R2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

Commit message: Motor encoder comparator setup
Parts:
- removed U? (x2): LM2903, symbol Comparator:LM2903
- added C5, C6: 0.1U, mini-mapper:C_0805, symbol mini-mapper:C
- added R13: 32K, mini-mapper:R_0805, symbol mini-mapper:R
- added R14: 1K, mini-mapper:R_0805, symbol mini-mapper:R
- added U3: LMV331, symbol mini-mapper:LMV331
- R10: renamed from R?; value CALC -> 100
- R12, R9: renamed from R?; value CALC -> 1K
- gave numbers to parts that had none: 8
- renumbered C3 to C4, J4 to J1, J1 to J2, J2 to J3, J3 to J4, NT1 to NT3, NT2 to NT4, R1 to R3, R2 to R4, R3 to R5, R4 to R6, R5 to R7, R6 to R8
Connections:
- net labels added: Vphoto
- wire segments 102 -> 121
Other:
- note added: "1. Does the current sense amplifier need input filters?\n\n2. Does the current sense amplifier need compensation?"
- note added: "3.3 V POWER FROM NUCLEO BOARD"
- note added: "Comparator hysteresis"
- note added: "Comparator threshold"
- note added: "Current: 0 ≤ I ≤ 250 mA\nKeep Vsense ≤ 100 mV\n\nRsense = 0.4 Ω ⇒ 0 ≤ Vsense ≤ 0.1 V\n\n(Pmax = 25 mW)\n"
- note added: "I(dark) = 100 nA (max.)\nI(light) = 1 mA (min.), 2 mA (typ.)"
- note added: "Infra-red LED"
- note added: "MOTOR POWER INPUT (4.5 V)"
- note added: "Motor coil\ncurrent sense\nopamp"
- note added: "Motor encoder\ncomparator"
- note added: "Phototransistor current"
- note added: "Phototransistor current conversion"
- note added: "R9 and R12 set the comparator threshold\nat Vcc/2 = 1.65 V. This is large enough to\navoid problems with ambient light "dark\ncurrent" from the phototransistor."
- note added: "To get Vphoto = 3.3 V for I(light) = 1 mA,\nput R11 = 3.3 kΩ\n\n(If I(light) > 1 mA, the phototransistor\njust goes into saturation anyway.)"
- note added: "Vf = 1.25 V (typ.), 1.6 V (max.)\nIf = 20 mA (nominal from datasheet plots)\n\nR10 = 100Ω ⇒ If = 20.5 mA (typ.), 17 mA (min.)"
- note added: "With comparator outputs 0 and 3.3 V,\nR14 = 1 kΩ, R13 = 32 kΩ gives\n\nV(hyst) = 1K/(1K + 32K) * (3.3 - 0) = 0.1 V"
- note removed: "1. Does the current sense amplifier need input filters?\n\n2. Does the current sense amplifier need compensation?\n\n3. What supply voltage for opamp and comparator?"
- note removed: "COPY TO PROJECT LIBRARY!"
- note removed: "Current: 0 ≤ I ≤ 250 mA\nKeep Vsense ≤ 100 mV\n\nRsense = 0.4 Ω ⇒\n 0 ≤ Vsense ≤ 0.1 V\n\n(Pmax = 25 mW)\n"
- note removed: "HYSTERESIS\n\nCOMPARATOR SELECTION\n\nCOMPARATOR POWER"
- note removed: "POWER"
- note removed: "POWER INPUT"
- moved on the sheet: J1, R10, R11, R12, R9, U2B, U4

Commit message: More on simulations; motor board power
Parts:
- removed J1: Conn_01x02, symbol mini-mapper:Conn_01x02
- added C? (x2): 1U, mini-mapper:C_0805, symbol mini-mapper:C
- added J?: Barrel_Jack, symbol mini-mapper:Barrel_Jack
- added TP?: TestPoint, TestPoint:TestPoint_Pad_2.0x2.0mm, symbol mini-mapper:TestPoint
- added U?: TLV70245_SOT23-5, Package_TO_SOT_SMD:SOT-23-5, symbol mini-mapper:TLV70245_SOT23-5
- R10: value 100 -> 82
- R11: value CALC -> 5.7K
Connections:
- wire segments 121 -> 135
Other:
- note added: "3.3V\nGND\nMOTOR_IN1\nMOTOR_IN2\nMOTOR_SENSE\nENCODER_PULSE"
- note added: "5V input"
- note added: "I(dark) = 100 nA (max.)\nI(light) = 1 mA (min.), 2 mA (typ.)\n\nBecause of geometry of overlap of holes\nin motor encoder disk with optical aperture,\nwe'll get 0.5 mA (min.), 1 mA (typ.)"
- note added: "MOTOR POWER INPUT (5V to 4.5 V)"
- note added: "NUCLEO CONNECTIONS"
- note added: "POWER"
- note added: "To get Vphoto high enough for I(light) = 0.5 mA,\nput R11 = 5.7 kΩ (gives Vphoto = 2.85 V)\n\n(If I(light) is much larger, the phototransistor\ngoes into saturation.)"
- note added: "Vf = 1.25 V (typ.), 1.6 V (max.)\nIf = 20 mA (nominal from datasheet plots)\n\nR10 = 82Ω ⇒ If = 25 mA (typ.), 21 mA (min.)"
- note removed: "I(dark) = 100 nA (max.)\nI(light) = 1 mA (min.), 2 mA (typ.)"
- note removed: "MOTOR POWER INPUT (4.5 V)"
- note removed: "To get Vphoto = 3.3 V for I(light) = 1 mA,\nput R11 = 3.3 kΩ\n\n(If I(light) > 1 mA, the phototransistor\njust goes into saturation anyway.)"
- note removed: "Vf = 1.25 V (typ.), 1.6 V (max.)\nIf = 20 mA (nominal from datasheet plots)\n\nR10 = 100Ω ⇒ If = 20.5 mA (typ.), 17 mA (min.)"
- moved on the sheet: C1, C2, C4, C5, C6, J2, J3, NT3, NT4, R10, R11, R12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

Commit message: Motor board schematic close to complete
Parts:
- removed C3: 100p, mini-mapper:C_0805, symbol mini-mapper:C
- removed J2: Conn_01x02, symbol mini-mapper:Conn_01x02
- removed J4, J5: Conn_01x01, symbol mini-mapper:Conn_01x01
- removed NT1, NT2: Net-Tie_2, symbol Device:Net-Tie_2
- removed R1, R2: 1K, mini-mapper:R_0805, symbol mini-mapper:R
- added J3: PinSocket_01x06, mini-mapper:PinSocket_1x06_P2.54mm_Vertical, symbol mini-mapper:PinSocket_01x06
- TP1: renamed from TP?; footprint TestPoint:TestPoint_Pad_2.0x2.0mm -> mini-mapper:TestPoint_Pad_2.0x2.0mm
- U1: renamed from U?; footprint Package_TO_SOT_SMD:SOT-23-5 -> mini-mapper:SOT-23-5
- gave numbers to parts that had none: 3
- renumbered C4 to C5, C5 to C6, C6 to C7, J3 to J2, NT3 to NT1, NT4 to NT2, R3 to R1, R4 to R2, R5 to R3, R6 to R4, R7 to R5, R8 to R6, R13 to R7, R9 to R8, R14 to R9, U1 to U2, U2 to U3, U3 to U4, U4 to U5
Connections:
- net labels added: ENCODER_PULSE, MOTOR_IN1, MOTOR_IN2, MOTOR_SENSE
- net labels removed: IN1, IN2, Vsense
Other:
- note added: "+3V3"
- note added: "ANALOG INPUT (PA3, ADC123_IN3)"
- note added: "CN7 16"
- note added: "CN7 18"
- note added: "CN8 11"
- note added: "CN8 16"
- note added: "CN8 7"
- note added: "CN9 1"
- note added: "DIGITAL INPUT (PG3)"
- note added: "DIGITAL OUTPUT (PD14, TIM4_CH3)"
- note added: "DIGITAL OUTPUT (PD15, TIM4_CH4)"
- note added: "Does the opamp U3A need compensation?"
- note added: "GND"
- note added: "Make sure the barrel jack is the right size and the "right way out"!"
- note added: "Make the Nucleo connection a header or a socket on the motor board?\nThe corresponding connector on the Nucleo board is a socket."
- note added: "NUCLEO PIN"
- note added: "OUTSTANDING ISSUES"
- note added: "R8 and R12 set the comparator threshold\nat Vcc/2 = 1.65 V. This is large enough to\navoid problems with ambient light "dark\ncurrent" from the phototransistor."
- note added: "With comparator outputs 0 and 3.3 V,\nR9 = 1 kΩ, R7 = 32 kΩ gives\n\nV(hyst) = 1K/(1K + 32K) * (3.3 - 0) = 0.1 V"
- note removed: "1. Does the current sense amplifier need input filters?\n\n2. Does the current sense amplifier need compensation?"
- note removed: "3.3V\nGND\nMOTOR_IN1\nMOTOR_IN2\nMOTOR_SENSE\nENCODER_PULSE"
- note removed: "Across\nsense\nresistor"
- note removed: "Example current sense amplifier input filter\n(from TI SLVA959A)"
- note removed: "QUESTIONS"
- note removed: "R9 and R12 set the comparator threshold\nat Vcc/2 = 1.65 V. This is large enough to\navoid problems with ambient light "dark\ncurrent" from the phototransistor."
- note removed: "To\nsense\namplifier"
- note removed: "With comparator outputs 0 and 3.3 V,\nR14 = 1 kΩ, R13 = 32 kΩ gives\n\nV(hyst) = 1K/(1K + 32K) * (3.3 - 0) = 0.1 V"

Commit message: Finish up motor board schematic; start on layout
Parts:
- removed J3: PinSocket_01x06, mini-mapper:PinSocket_1x06_P2.54mm_Vertical, symbol mini-mapper:PinSocket_01x06
- removed NT1, NT2: Net-Tie_2, symbol Device:Net-Tie_2
- added J3: PinHeader_01x06, mini-mapper:PinHeader_1x06_P2.54mm_Vertical, symbol mini-mapper:PinHeader_01x06
- C1: footprint (none) -> mini-mapper:CP_Elec_6.3x7.7; MPN (none) -> EEE-HC1C101XP
- J1: value Barrel_Jack -> PJ-063AH; footprint (none) -> mini-mapper:BarrelJack_CUI_PJ-063AH_Horizontal; MPN (none) -> PJ-063AH
- J2: footprint (none) -> mini-mapper:PinSocket_1x02_P2.54mm_Vertical; MPN (none) -> SLW-102-01-T-S
- TP1: MPN (none) -> n/a
- U1: MPN (none) -> TLV70245DBVR
- U3: MPN (none) -> TLV9051IDBVR
- U4: footprint (none) -> mini-mapper:SOT-23-5; MPN (none) -> LMV331IDBVR
- U5: footprint (none) -> mini-mapper:TCST1202; MPN (none) -> TCST1202
Connections:
- net Isense- is gone; now on net GND: R3.1, R6.1
- net +3V3: now also J3.1 (Pin_1)
- net ENCODER_PULSE: now also J3.2 (Pin_2)
- net GND: now also J3.6 (Pin_6)
- net Isense+: now also R2.1, U2.7 (RS)
- net MOTOR_IN1: now also J3.4 (Pin_4)
- net MOTOR_IN2: now also J3.5 (Pin_5)
- net MOTOR_SENSE: now also J3.3 (Pin_3)
Other:
- note added: "f(PWM) = 31.25 kHz"
- note removed: "Does the opamp U3A need compensation?"
- note removed: "Make sure the barrel jack is the right size and the "right way out"!"
- note removed: "Make the Nucleo connection a header or a socket on the motor board?\nThe corresponding connector on the Nucleo board is a socket."
- note removed: "OUTSTANDING ISSUES"
Changed lines of the file:
@@
 Comment1 "Designed for AISLER 2-Layer Service"
 Comment2 "Part of the Mini-Mapper project"
-Comment3 ""
+Comment3 "Motor driver and encoder prototype board"
 Comment4 ""
 $EndDescr
@@
 Wire Wire Line
 	3450 1025 3450 1075
-Wire Wire Line
-	1450 1750 3050 1750
-Wire Wire Line
-	3050 1850 1450 1850
 $Comp
 L mini-mapper:C C2
@@
 F 0 "C1" H 2443 1321 50  0000 L CNN
 F 1 "100U" H 2443 1230 50  0000 L CNN
-F 2 "" H 2363 1125 50  0001 C CNN
-F 3 "~" H 2325 1275 50  0001 C CNN
+F 2 "mini-mapper:CP_Elec_6.3x7.7" H 2363 1125 50  0001 C CNN
+F 3 "https://www.mouser.at/datasheet/2/315/ABA0000C1160-947462.pdf" H 2325 1275 50  0001 C CNN
+F 4 "EEE-HC1C101XP" H 2325 1275 50  0001 C CNN "MPN"
 	1    2325 1275
 	1    0    0    -1
@@
 Text Notes 7975 1225 0    50   ~ 10
 MOTOR POWER INPUT (5V to 4.5 V)
-Text Notes 1025 1400 0    50   ~ 10
+Text Notes 900  1450 0    50   ~ 10
 CONTROL INPUT
 Text Label 2650 2100 0    50   ~ 0
@@
 F 2 "mini-mapper:SOT-23-5" H 8625 3175 50  0001 C CNN
 F 3 "https://www.ti.com/lit/ds/symlink/tlv9052.pdf" H 8625 3175 50  0001 C CNN
+F 4 "TLV9051IDBVR" H 8625 3175 50  0001 C CNN "MPN"
 	2    8625 3175
 	1    0    0    -1
@@
 Text Notes 6575 2175 0    50   ~ 10
 CURRENT SENSE OUTPUT
-Text Label 1450 1750 0    50   ~ 0
+Text Label 1025 1750 0    50   ~ 0
 MOTOR_IN1
-Text Label 1450 1850 0    50   ~ 0
+Text Label 1025 1850 0    50   ~ 0
 MOTOR_IN2
 Text Label 6750 2350 0    50   ~ 0
@@
 F 0 "J2" H 4168 1525 50  0000 C CNN
 F 1 "Conn_01x02" H 4168 1616 50  0000 C CNN
-F 2 "" H 4250 1850 50  0001 C CNN
-F 3 "~" H 4250 1850 50  0001 C CNN
+F 2 "mini-mapper:PinSocket_1x02_P2.54mm_Vertical" H 4250 1850 50  0001 C CNN
+F 3 "https://www.mouser.at/datasheet/2/527/slw-1370256.pdf" H 4250 1850 50  0001 C CNN
+F 4 "SLW-102-01-T-S" H 4250 1850 50  0001 C CNN "MPN"
 	1    4250 1850
 	1    0    0    1
@@
 Text Notes 6550 2700 0    50   Italic 10
 Current sense amplifier
-$Comp
-L Device:Net-Tie_2 NT1
-U 1 1 5F094D37
-P 3875 2325
-F 0 "NT1" H 3875 2450 50  0000 C CNN
-F 1 "Net-Tie_2" H 3950 2375 50  0000 C CNN
-F 2 "" H 3875 2325 50  0001 C CNN
-F 3 "~" H 3875 2325 50  0001 C CNN
-	1    3875 2325
-	1    0    0    -1
-$EndComp
-$Comp
-L Device:Net-Tie_2 NT2
-U 1 1 5F09CC8D
-P 3875 2700
-F 0 "NT2" H 3875 2575 50  0000 C CNN
-F 1 "Net-Tie_2" H 3950 2650 50  0000 C CNN
-F 2 "" H 3875 2700 50  0001 C CNN
-F 3 "~" H 3875 2700 50  0001 C CNN
-	1    3875 2700
-	1    0    0    -1
-$EndComp
 Wire Wire Line
 	3650 2300 3650 2325
-Wire Wire Line
-	3775 2325 3650 2325
 Connection ~ 3650 2325
 Wire Wire Line
@@
 Wire Wire Line
 	3650 2675 3650 2700
-Wire Wire Line
-	3775 2700 3650 2700
 Connection ~ 3650 2700
 Wire Wire Line
@@
 F 0 "U5" H 1225 6100 50  0000 C CNN
 F 1 "TCST1202" H 1225 6009 50  0000 C CNN
-F 2 "" H 1225 5675 50  0001 C CNN
-F 3 "" H 1225 5675 50  0001 C CNN
+F 2 "mini-mapper:TCST1202" H 1225 5675 50  0001 C CNN
+F 3 "https://www.vishay.com/docs/83764/tcst1103.pdf" H 1225 5675 50  0001 C CNN
+F 4 "TCST1202" H 1225 5675 50  0001 C CNN "MPN"
 	1    1225 5675
 	1    0    0    -1
@@
 F 0 "U4" H 3675 6240 50  0000 C CNN
 F 1 "LMV331" H 3675 6149 50  0000 C CNN
-F 2 "" H 3675 5975 50  0001 C CNN
+F 2 "mini-mapper:SOT-23-5" H 3675 5975 50  0001 C CNN
 F 3 "http://www.ti.com/lit/ds/symlink/lmv331.pdf" H 3675 6075 50  0001 C CNN
+F 4 "LMV331IDBVR" H 3575 5875 50  0001 C CNN "MPN"
 	1    3575 5875
 	1    0    0    -1
@@
 F 0 "U4" H 9700 3225 50  0000 L CNN
 F 1 "LMV331" H 9700 3125 50  0000 L CNN
-F 2 "" H 9675 3275 50  0001 C CNN
+F 2 "mini-mapper:SOT-23-5" H 9675 3275 50  0001 C CNN
 F 3 "http://www.ti.com/lit/ds/symlink/lmv331.pdf" H 9675 3375 50  0001 C CNN
+F 4 "LMV331IDBVR" H 9575 3175 50  0001 C CNN "MPN"
 	2    9575 3175
 	1    0    0    -1
@@
 F 1 "TestPoint" H 1958 5652 50  0000 L CNN
 F 2 "mini-mapper:TestPoint_Pad_2.0x2.0mm" H 2100 5625 50  0001 C CNN
-F 3 "~" H 2100 5625 50  0001 C CNN
+F 3 "n/a" H 2100 5625 50  0001 C CNN
+F 4 "n/a" H 1900 5625 50  0001 C CNN "MPN"
 	1    1900 5625
 	1    0    0    -1
@@
 P 8575 1675
 F 0 "J1" H 8632 2000 50  0000 C CNN
-F 1 "Barrel_Jack" H 8632 1909 50  0000 C CNN
-F 2 "" H 8625 1635 50  0001 C CNN
-F 3 "~" H 8625 1635 50  0001 C CNN
+F 1 "PJ-063AH" H 8632 1909 50  0000 C CNN
+F 2 "mini-mapper:BarrelJack_CUI_PJ-063AH_Horizontal" H 8625 1635 50  0001 C CNN
+F 3 "https://www.mouser.at/datasheet/2/670/pj-063ah-1778660.pdf" H 8625 1635 50  0001 C CNN
+F 4 "PJ-063AH" H 8575 1675 50  0001 C CNN "MPN"
 	1    8575 1675
 	1    0    0    -1
@@
 F 2 "mini-mapper:SOT-23-5" H 9825 2000 50  0001 C CIN
 F 3 "http://www.ti.com/lit/ds/symlink/tlv702.pdf" H 9825 1725 50  0001 C CNN
+F 4 "TLV70245DBVR" H 9825 1675 50  0001 C CNN "MPN"
 	1    9825 1675
 	1    0    0    -1
@@
 ENCODER_PULSE
 $Comp
-L mini-mapper:PinSocket_01x06 J3
-U 1 1 5F1B572A
-P 8700 5425
-F 0 "J3" H 8750 4975 50  0000 L CNN
-F 1 "PinSocket_01x06" H 8750 4875 50  0000 L CNN
-F 2 "mini-mapper:PinSocket_1x06_P2.54mm_Vertical" H 8700 5425 50  0001 C CNN
-F 3 "~" H 8700 5425 50  0001 C CNN
-	1    8700 5425
-	1    0    0    -1
-$EndComp
-$Comp
 L power:+3V3 #PWR017
 U 1 1 5F1BF659
@@
 Wire Wire Line
 	8500 5425 7450 5425
+Text Label 7450 5525 0    50   ~ 0
+MOTOR_IN1
+Text Label 7450 5625 0    50   ~ 0
+MOTOR_IN2
+Wire Wire Line
+	8500 5525 7450 5525
+Wire Wire Line
+	8500 5625 7450 5625
+Text Label 7450 5425 0    50   ~ 0
+MOTOR_SENSE
 Text Label 7450 5325 0    50   ~ 0
-MOTOR_IN1
-Text Label 7450 5425 0    50   ~ 0
-MOTOR_IN2
-Wire Wire Line
-	8500 5525 7450 5525
-Wire Wire Line
-	8500 5625 7450 5625
-Text Label 7450 5525 0    50   ~ 0
-MOTOR_SENSE
-Text Label 7450 5625 0    50   ~ 0
 ENCODER_PULSE
 Text Notes 8850 5250 0    50   ~ 0
@@
 Text Notes 8850 5750 0    50   ~ 0
 GND
+Text Notes 8850 5550 0    50   ~ 0
+DIGITAL OUTPUT (PD14, TIM4_CH3)
+Text Notes 8850 5650 0    50   ~ 0
+DIGITAL OUTPUT (PD15, TIM4_CH4)
+Text Notes 8850 5450 0    50   ~ 0
+ANALOG INPUT (PA3, ADC123_IN3)
 Text Notes 8850 5350 0    50   ~ 0
-DIGITAL OUTPUT (PD14, TIM4_CH3)
-Text Notes 8850 5450 0    50   ~ 0
-DIGITAL OUTPUT (PD15, TIM4_CH4)
-Text Notes 8850 5550 0    50   ~ 0
-ANALOG INPUT (PA3, ADC123_IN3)
-Text Notes 8850 5650 0    50   ~ 0
 DIGITAL INPUT (PG3)
 Text Notes 8850 5125 0    75   ~ 15
 NUCLEO PIN
-Text Notes 12100 1150 0    100  ~ 0
-Does the opamp U3A need compensation?
 Wire Wire Line
 	10300 1575 10625 1575
@@
 Wire Wire Line
 	8400 5150 8400 5225
-Text Notes 12100 1550 0    100  ~ 0
-Make sure the barrel jack is the right size and the "right way out"!
-Text Notes 12100 2050 0    100  ~ 0
-Make the Nucleo connection a header or a socket on the motor board?\nThe corresponding connector on the Nucleo board is a socket.
-Text Notes 10275 5275 0    50   ~ 0
+Text Notes 10275 5250 0    50   ~ 0
 CN8  7
-Text Notes 10275 5775 0    50   ~ 0
+Text Notes 10275 5750 0    50   ~ 0
 CN8 11
-Text Notes 10275 5375 0    50   ~ 0
+Text Notes 10275 5550 0    50   ~ 0
 CN7 16
-Text Notes 10275 5475 0    50   ~ 0
+Text Notes 10275 5650 0    50   ~ 0
 CN7 18
-Text Notes 10275 5575 0    50   ~ 0
+Text Notes 10275 5450 0    50   ~ 0
 CN9  1
-Text Notes 10275 5675 0    50   ~ 0
+Text Notes 10275 5350 0    50   ~ 0
 CN8 16
-Text Notes 12125 825  0    100  ~ 20
-OUTSTANDING ISSUES
+$Comp
+L mini-mapper:PinHeader_01x06 J3
+U 1 1 5F1C4768
+P 8700 5425
+F 0 "J3" H 8700 5000 50  0000 L CNN
+F 1 "PinHeader_01x06" H 8700 4900 50  0000 L CNN
+F 2 "mini-mapper:PinHeader_1x06_P2.54mm_Vertical" H 8700 5425 50  0001 C CNN
+F 3 "https://www.mouser.at/datasheet/2/276/0022284060_PCB_HEADERS-228129.pdf" H 8700 5425 50  0001 C CNN
+F 4 "22-28-4060" H 8700 5425 50  0001 C CNN "MPN"
+	1    8700 5425
+	1    0    0    -1
+$EndComp
+Wire Wire Line
+	3650 2325 3975 2325
+Wire Wire Line
+	3650 2700 3975 2700
+Text Notes 825  1575 0    50   ~ 0
+f(PWM) = 31.25 kHz
+Wire Wire Line
+	1025 1750 3050 1750
+Wire Wire Line
+	1025 1850 3050 1850
 $EndSCHEMATC

Commit message: Missed some changes...
Parts:
- added H1, H2, H3, H4: MountingHole, mini-mapper:MountingHole_2.7mm_M2.5, symbol mini-mapper:MountingHole
- C2, C5, C6, C7: MPN (none) -> 885012207098
- C3, C4: MPN (none) -> 885012107015
- R1: value 7K -> 56K; MPN (none) -> CRGP0805F56K
- R10: MPN (none) -> CRCW080582R0FKEA
- R11: value 5.7K -> 5.6K; MPN (none) -> CRCW08055K60FKEAC
- R12, R8: MPN (none) -> CRGP0805F1K0
- R2: MPN (none) -> RL0805FR-070R4L
- R3: MPN (none) -> CRCW080512K0FKEA
- R4: value 2K -> 16K; MPN (none) -> CRCW080516K0FKEA
- R5: MPN (none) -> CRCW0805330KFKEA
- R6: MPN (none) -> CRGP0805F220K
- R7: value 32K -> 240K; MPN (none) -> CRCW0805240KFKEA
- R9: value 1K -> 7.5K; MPN (none) -> CRCW08057K50FKEA
Connections:
- net MOTOR_IN1: now also J3.3 (Pin_3); no longer J3.4 (Pin_4)
- net MOTOR_IN2: now also J3.4 (Pin_4); no longer J3.5 (Pin_5)
- net MOTOR_SENSE: now also J3.5 (Pin_5); no longer J3.3 (Pin_3)
- net MOTOR2: now reaches J2.2 (Pin_2), U2.6 (OUT1)
- net MOTOR1: now reaches J2.1 (Pin_1), U2.8 (OUT2)
- net VIN: now reaches C3.1, J1.1, U1.1 (IN), U1.3 (EN)
Other:
- note added: "To get Vphoto high enough for I(light) = 0.5 mA,\nput R11 = 5.6 kΩ (gives Vphoto = 2.8 V)\n\n(If I(light) is much larger, the phototransistor\ngoes into saturation.)"
- note added: "With comparator outputs 0 and 3.3 V,\nR9 = 7.5 kΩ, R7 = 240 kΩ gives\n\nV(hyst) = 7.5K/(7.5K + 240K) * (3.3 - 0) = 0.1 V"
- note removed: "To get Vphoto high enough for I(light) = 0.5 mA,\nput R11 = 5.7 kΩ (gives Vphoto = 2.85 V)\n\n(If I(light) is much larger, the phototransistor\ngoes into saturation.)"
- note removed: "With comparator outputs 0 and 3.3 V,\nR9 = 1 kΩ, R7 = 32 kΩ gives\n\nV(hyst) = 1K/(1K + 32K) * (3.3 - 0) = 0.1 V"
- moved on the sheet: J2
